Commit message: changes

File: carsim_discription/urdf/model.urdf (robot description, URDF)
Before this commit: robot basic_car, 8 links, 7 joints
Joints:
- joint left_wheel_hinge: limit effort=100 velocity=6.0 -> effort=100 velocity=100.0
- joint right_wheel_hinge: limit effort=100 velocity=6.0 -> effort=100 velocity=100.0

Commit message: basic changes

File: carsim_discription/urdf/model.urdf (robot description, URDF)
Before this commit: robot basic_car, 8 links, 7 joints
Links:
- link base_link: mass 10 -> 0.5

Commit message: cleaning

File: carsim_discription/urdf/model.urdf (robot description, URDF)
Before this commit: robot basic_car, 8 links, 7 joints
Links:
- link base_link: mass 0.5 -> 1
